File: KiCad/projet_capteur_lebon/projet_capteur_lebon.kicad_pcb (KiCad board)
At the start: 2 copper layers, 68.6 x 53.3 mm, 8 parts, among them J1 Power, J2 Digital/PWM, J3 Analog, J4 Digital/PWM

Commit message: Création symbole + empreinte OLED
Parts:
- added U1: ~, librairie_empreintes:SIP-4, F.Cu at (166.0, 78.3)
