File: KiCad/projet_capteur_lebon/projet_capteur_lebon.kicad_sch (KiCad schematic)
At the start: 17 parts, among them J1 Power, J2 Digital/PWM, J3 Analog, J4 Digital/PWM

Commit message: Etiquette
Parts:
- added C3: c, librairie_empreintes:C_Disc_D6.0mm_W2.5mm_P5.00mm, symbol Device:C
Connections:
- net +5V: no longer U5. (2)
- net GND: now also U3.3 (GND), C3.2; no longer U3.4 (TXD)
- net BT 1: now reaches U3.1 (EN)
- net 5V: now reaches U3.2 (VCC)
- net 5V: now also U1.2 (VCC), U2.4 (VCC), U5. (2)
- net EROT 1: now reaches U2.1 (CLK)
- net EROT 1: now also C3.1
- net EROT 2: now reaches U2.2 (DT)
- net EROT 3: now reaches U2.3 (SW)
- net OLED 3: now reaches U1.3 (SCL)
- net OLED 4: now reaches U1.4 (SDA)
- new net BT 4: U3.4 (TXD)
Other:
- moved on the sheet: R2
